File: sch/alim.kicad_sch (KiCad schematic)
At the start: 4 parts, among them J1 PWR

Commit message: alim / core
Signed-off-by: cukier <mauriciocukier@gmail.com>
Parts:
- added C1: 470uF, Capacitor_THT:CP_Radial_D12.5mm_P5.00mm, symbol Device:C_Polarized
- added C2, C6: 1000uF, Capacitor_THT:CP_Radial_D8.0mm_P3.50mm, symbol Device:C_Polarized
- added C3, C4, C5: 100nF, Capacitor_SMD:C_0805_2012Metric, symbol Device:C
- added D2, D3: US1M, Diode_SMD:D_SMA, symbol Diode:US1M
- added D4: PWR, LED_SMD:LED_0805_2012Metric, symbol Device:LED
- added R2: 1k, Resistor_SMD:R_0805_2012Metric, symbol Device:R
- added U1: uA7805, Package_TO_SOT_SMD:TO-263-2, symbol Regulator_Linear:uA7805
- added U2: AMS1117-3.3, Package_TO_SOT_SMD:SOT-223-3_TabPin2, symbol Regulator_Linear:AMS1117-3.3
- R1: footprint (none) -> Varistor:RV_Disc_D12mm_W4.5mm_P7.5mm
Connections:
- net GND: now also C1.2, C2.2, C3.2, C4.2, C5.2, C6.2, D4.1 (K), U1.2 (GND), U2.1 (GND)
- net at D1.1 (K): now also C1.1, C3.1, D2.1 (K), U1.1 (IN)
- net +24V: now reaches D1.2 (A), F1.2, R1.1
- new net: D4.2 (A), R2.2
- new net +3V3: C5.1, C6.1, D3.2 (A), U2.2 (VO)
- new net +5V: C2.1, C4.1, D2.2 (A), D3.1 (K), R2.1, U1.3 (OUT), U2.3 (VI)
Other:
- moved on the sheet: D1, F1, J1, R1
