File: sch/Nautilus.kicad_sch (KiCad schematic)
At the start: 0 parts

Commit message: alim / core
Signed-off-by: cukier <mauriciocukier@gmail.com>
Other:
- added sheet core (core.kicad_sch)
Changed lines of the file:
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@@
 	(paper "A4")
 	(sheet
+		(at 85.09 68.58)
+		(size 58.42 41.275)
+		(fields_autoplaced yes)
+		(stroke
+			(width 0.1524)
+			(type solid)
+			(color 72 0 0 1)
+		)
+		(fill
+			(color 255 255 194 1.0000)
+		)
+		(property "Sheetname" "core"
+			(at 85.09 67.8684 0)
+			(effects
+				(font
+					(size 1.27 1.27)
+				)
+				(justify left bottom)
+			)
+		)
+		(property "Sheetfile" "core.kicad_sch"
+			(at 85.09 110.4396 0)
+			(effects
+				(font
+					(size 1.27 1.27)
+				)
+				(justify left top)
+			)
+		)
+		(instances
+			(project "Nautilus"
+				(path "/923bbe6b-84fc-4c9c-ba1b-9f61307feb8d"
+					(page "3")
+				)
+			)
+		)
+	)
+	(sheet
 		(at 85.09 46.99)
-		(size 44.45 33.655)
+		(size 12.7 3.81)
 		(fields_autoplaced yes)
 		(stroke
@@
 		)
 		(property "Sheetfile" "alim.kicad_sch"
-			(at 85.09 81.2296 0)
+			(at 85.09 51.3846 0)
 			(effects
 				(font

Commit message: led driver
Signed-off-by: cukier <mauriciocukier@gmail.com>
Other:
- added sheet chan (chan.kicad_sch)
- sheet core ports: added CHAN_1, CHAN_2, CHAN_3, FAN; removed none
Changed lines of the file:
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@@
 	(sheet
 		(at 85.09 68.58)
-		(size 58.42 41.275)
+		(size 12.7 10.16)
 		(fields_autoplaced yes)
 		(stroke
@@
 		)
 		(property "Sheetfile" "core.kicad_sch"
-			(at 85.09 110.4396 0)
+			(at 85.09 79.3246 0)
 			(effects
 				(font
@@
 				)
 				(justify left top)
+			)
+		)
+		(pin "CHAN_1" input
+			(at 97.79 69.85 0)
+			(effects
+				(font
+					(size 1.27 1.27)
+				)
+				(justify right)
+			)
+		)
+		(pin "FAN" input
+			(at 97.79 77.47 0)
+			(effects
+				(font
+					(size 1.27 1.27)
+				)
+				(justify right)
+			)
+		)
+		(pin "CHAN_2" input
+			(at 97.79 72.39 0)
+			(effects
+				(font
+					(size 1.27 1.27)
+				)
+				(justify right)
+			)
+		)
+		(pin "CHAN_3" input
+			(at 97.79 74.93 0)
+			(effects
+				(font
+					(size 1.27 1.27)
+				)
+				(justify right)
 			)
 		)
@@
 				)
 			)
+		)
+	)
+	(sheet
+		(at 115.57 70.485)
+		(size 15.24 10.16)
+		(fields_autoplaced yes)
+		(stroke
+			(width 0.1524)
+			(type solid)
+			(color 72 0 0 1)
+		)
+		(fill
+			(color 255 255 194 1.0000)
+		)
+		(property "Sheetname" "chan"
+			(at 115.57 69.7734 0)
+			(effects
+				(font
+					(size 1.27 1.27)
+				)
+				(justify left bottom)
+			)
+		)
+		(property "Sheetfile" "chan.kicad_sch"
+			(at 115.57 81.2296 0)
+			(effects
+				(font
+					(size 1.27 1.27)
+				)
+				(justify left top)
+			)
+		)
+		(instances
+			(project "Nautilus"
+				(path "/923bbe6b-84fc-4c9c-ba1b-9f61307feb8d"
+					(page "4")
+				)
+			)
