File: sch/core.kicad_sch (KiCad schematic)
At the start: 10 parts, among them J2 PROG, Q2 MMBT2222A, Q3 MMBT2222A, U3 ESP32-WROOM-32

Commit message: led driver
Signed-off-by: cukier <mauriciocukier@gmail.com>
Parts:
- added D5: RX, LED_SMD:LED_0805_2012Metric, symbol Device:LED
- added D6: Tx, LED_SMD:LED_0805_2012Metric, symbol Device:LED
- added R5, R8: 1k, Resistor_SMD:R_0805_2012Metric, symbol Device:R
Connections:
- net GND: now also D5.1 (K), D6.1 (K)
- net RX: now also R8.2
- net TX: now also R5.2
- new net: D5.2 (A), R8.1
- new net: D6.2 (A), R5.1
